File: 01_Hardware/ATU-FT891/ATU-FT891.kicad_sch (KiCad schematic)
At the start: 25 parts

Commit message: first schematic
Parts:
- removed U?: ATmega328-P, Package_DIP:DIP-28_W7.62mm, symbol MCU_Microchip_ATmega:ATmega328-P
- added C? (x19): 100n, symbol Device:C
- added C? (x4): 10uF, symbol Device:C_Polarized
- added C? (x2): 10u, symbol Device:C
- added C? (x6): C, symbol Device:C
- added C? (x6): 100nF, symbol Device:C
- added C? (x3): 100uF, symbol Device:C_Polarized
- added D?: >2.5, symbol Device:LED
- added D?: <2.5, symbol Device:LED
- added D? (x14): 1N4148W, Diode_SMD:D_SOD-123, symbol Diode:1N4148W
- added D? (x2): D_Schottky, symbol Device:D_Schottky
- added D?: LNA, symbol Device:LED
- added D?: ACT, symbol Device:LED
- added D?: <2.0, symbol Device:LED
- added D?: <1.5, symbol Device:LED
- added F? (x2): Polyfuse, symbol Device:Polyfuse
- added J?: Mini-DIN-8, symbol Connector:Mini-DIN-8
- added J? (x3): Conn_Coaxial, symbol Connector:Conn_Coaxial
- added J?: Mini-DIN-6, symbol Connector:Mini-DIN-6
- added J? (x2): USB_B, symbol Connector:USB_B
- added J?: Conn_01x03_Male, symbol Connector:Conn_01x03_Male
- added JP? (x2): SolderJumper_2_Open, symbol Jumper:SolderJumper_2_Open
- added K? (x2): G5V-1, Relay_THT:Relay_SPDT_Omron_G5V-1, symbol Relay:G5V-1
- added L? (x2): 100u, symbol Device:L_Ferrite
- added LNA: 0, symbol Device:R
- added Q? (x18): 2N2222A_SMD, Package_TO_SOT_SMD:TSOT-23, symbol Transistor:2N2222A_SMD
- added R? (x5): R, symbol Device:R
- added R? (x20): 10k, symbol Device:R
- added R? (x14): 100k, symbol Device:R
- added R? (x2): 1k, symbol Device:R
- added SW?: TUNE, symbol Switch:SW_Push
- added SW?: LNA, symbol Switch:SW_Push
- added SW?: RST, symbol Switch:SW_Push
- added U?: Pico, RPi_Pico:RPi_Pico_SMD_TH, symbol RPi:Pico
- added U?: CM118B, Package_QFP:LQFP-48_7x7mm_P0.5mm, symbol CM118B:CM118B
- added U?: SL2.1A, SO16, symbol SL2.1:SL2.1A
- added U?: NCP1117-3.3_SOT223, Package_TO_SOT_SMD:SOT-223-3_TabPin2, symbol Regulator_Linear:NCP1117-3.3_SOT223
- added U?: NCP1117-5.0_SOT223, Package_TO_SOT_SMD:SOT-223-3_TabPin2, symbol Regulator_Linear:NCP1117-5.0_SOT223
- added Y?: Crystal, symbol Device:Crystal
- C?: value C -> 10pF
- C?: value C -> 22pF
- C?: value C -> 220pF
- C?: value C -> 47pF
- C?: value C -> 100pF
- L?: value L_Iron -> 2.2uH
- L?: value L_Iron -> 1uH
- L?: value L_Iron -> 0.05uH
- L?: value L_Iron -> 0.1uH
- L?: value L_Iron -> 0.47uH
- L?: value L_Iron -> 0.22uH
Connections:
- net +12V: now also C?.1, C?.1, C?.1, C?.1, C?.1, C?.1, C?.1, C?.1, C?.1, C?.1, C?.1, C?.1, C?.1, C?.1, D?.1 (K), D?.1 (K), D?.1 (K), D?.1 (K), D?.1 (K), D?.1 (K), D?.1 (K), D?.1 (K), D?.1 (K), D?.1 (K), D?.1 (K), D?.1 (K), D?.1 (K), D?.1 (K), J?.1, K?.2, K?.2
- net C1_OC: now also C?.2, D?.2 (A), Q?.3 (C)
- net C2_OC: now also C?.2, D?.2 (A), Q?.3 (C)
- net C3_OC: now also C?.2, D?.2 (A), Q?.3 (C)
- net C4_OC: now also C?.2, D?.2 (A), Q?.3 (C)
- net C5_OC: now also C?.2, D?.2 (A), Q?.3 (C)
- net IO_OC: now also C?.2, D?.2 (A), Q?.3 (C)
- net L1_I: now also K?.1
- net L1_OC: now also C?.2, D?.2 (A), Q?.3 (C)
- net L2_OC: now also C?.2, D?.2 (A), Q?.3 (C)
- net L3_OC: now also C?.2, D?.2 (A), Q?.3 (C)
- net L4_OC: now also C?.2, D?.2 (A), Q?.3 (C)
- net L5_OC: now also C?.2, D?.2 (A), Q?.3 (C)
- net L6_OC: now also C?.2, D?.2 (A), Q?.3 (C)
- net SDR_OUT: now also K?.1, J?.1 (In); no longer K?.10
- net GND renamed AVSS
- net AVSS: now also C?.2, C?.2, C?.2, C?.2, C?.2, C?.2, C?.2, C?.2, C?.2, C?.2, C?.2, C?.2, C?.2, C?.2, C?.2, C?.2, C?.2, C?.2, C?.2, C?.2, C?.2, C?.2, D?.1 (K), D?.1 (K), D?.1 (K), D?.1 (K), D?.1 (K), J?.2, J?.2 (Ext), J?.2 (Ext), J?.2 (Ext), J?.3, J?.4 (GND), J?.4 (GND), J?.5 (Shield), J?.5 (Shield), JP?.1 (A), Q?.2 (E), Q?.2 (E), Q?.2 (E), Q?.2 (E), Q?.2 (E), Q?.2 (E), Q?.2 (E), Q?.2 (E), Q?.2 (E), Q?.2 (E), Q?.2 (E), Q?.2 (E), Q?.2 (E), Q?.2 (E), Q?.2 (E), Q?.2 (E), Q?.2 (E), R?.2, R?.2, R?.2, R?.2, R?.2, R?.2, R?.2, R?.2, R?.2, R?.2, R?.2, R?.2, R?.2, R?.2, SW?.1, SW?.1, SW?.1, U?.1 (GND), U?.1 (GND), U?.12 (GND), U?.13 (GND), U?.13 (MODE), U?.15 (DVSS), U?.18 (GND), U?.21 (TEST), U?.22 (AVSS), U?.23 (GND), U?.28 (GND), U?.3 (GND), U?.32 (AVSS), U?.33 (AGND), U?.35 (DVSS), U?.38 (GND), U?.8 (GND)
- net L6_O renamed ANT_OUT
- net ANT_OUT: now also J?.1 (In)
- net PAN renamed TX
- net TX: now also C?.2, D?.2 (A), Q?.3 (C)
- net SDR_IN renamed RF_IN
- net RF_IN: now also J?.1 (In), K?.5, K?.6
- new net: D?.2 (A), R?.2 (x6)
- new net: JP?.2 (B), JP?.2 (B), U?.39 (MSEL)
- new net: Q?.1 (B), R?.1, R?.1 (x13)
- new net: D?.1 (K), F?.2 (x2)
- new net: C?.1, U?.37 (DREG18)
- new net: C?.1, U?.14 (VDD18)
- new net: K?.10, LNA.1
- new net: K?.10, LNA.2
- new net: C?.1, U?.31 (LOR)
- new net: J?.1 (Pin_1), U?.41 (SWCLK)
- new net: J?.2 (Pin_2), U?.42 (GND)
- new net: J?.3 (Pin_3), U?.43 (SWDIO)
- new net: C?.1, U?.29 (LOL)
- new net: C?.1, C?.1, U?.3 (VI) (x2)
- new net: C?.2, U?.25 (MICINL)
- new net: Q?.1 (B), Q?.3 (C), R?.2
- new net: K?.1, K?.1
- new net: C?.1, U?.42 (DREG33)
- new net: Q?.1 (B), Q?.3 (C), R?.1, R?.2
- new net: C?.2, U?.27 (MICINR)
- new net: U?.43 (USBDP), U?.6 (DP2)
- new net: U?.44 (USBDM), U?.5 (DM2)
- new net: D?.1 (K), Q?.3 (C)
- new net: Q?.1 (B), R?.2 (x2)
- new net: Q?.2 (E), Q?.3 (C)
- new net: C?.1, U?.13 (VDD33)
- new net: J?.2 (D-), U?.7 (DM1)
- new net: J?.3 (D+), U?.8 (DP1)
- new net: U?.16 (XIN), Y?.1
- new net: U?.15 (XOUT), Y?.2
- new net: J?.3 (D+), U?.10 (DP)
- new net: J?.2 (D-), U?.9 (DM)
- new net +3.3V: C?.1, C?.1, C?.1, JP?.1 (A), L?.1, R?.1, R?.1, R?.1, R?.1, R?.1, R?.1, R?.1, R?.2, U?.10 (PWRSEL), U?.2 (VO), U?.36 (3V3), U?.38 (MICONLY)
- new net +3.3VA: C?.1, L?.2, U?.35 (ADC_VREF), U?.36 (AREG36)
- new net +5P: C?.1, C?.1, C?.1, D?.2 (A), D?.2 (A), J?.1 (VBUS), J?.1 (VBUS)
- new net +5V: C?.1, C?.1, C?.1, C?.1, F?.1, F?.1, L?.1, U?.11 (VDD5), U?.2 (VO), U?.34 (DVDD)
- new net +5VA: C?.1, C?.1, C?.1, L?.2, U?.28 (AVDD), U?.33 (AVDD)
- new net C1+: R?.2, U?.11 (GPIO8)
- new net C2+: R?.2, U?.12 (GPIO9)
- new net C3+: R?.2, U?.14 (GPIO10)
- new net C4+: R?.2, U?.15 (GPIO11)
- new net C5+: R?.2, U?.16 (GPIO12)
- new net DAT_IN: C?.2, C?.2, J?.1
- new net DAT_OUT: C?.1, C?.1, J?.5
- new net FWD: U?.31 (GPIO26_ADC0)
- new net IO+: R?.2, U?.17 (GPIO13)
- new net L1+: R?.2, U?.4 (GPIO2)
- new net L2+: R?.2, U?.5 (GPIO3)
- new net L3+: R?.2, U?.6 (GPIO4)
- new net L4+: R?.2, U?.7 (GPIO5)
- new net L5+: R?.2, U?.9 (GPIO6)
- new net L6+: R?.2, U?.10 (GPIO7)
- new net LNA_: R?.2, SW?.2, U?.21 (GPIO16)
- new net LNA_SW: R?.1, R?.1, U?.19 (GPIO14)
- new net LNA_TR: C?.2, D?.2 (A), K?.9, K?.9, Q?.3 (C)
- new net REV: U?.32 (GPIO27_ADC1)
- new net RST: R?.2, SW?.2, U?.30 (RUN)
- new net RX0: U?.2 (GPIO1)
- new net SWR1: R?.1, U?.20 (GPIO15)
- new net SWR2: R?.1, U?.34 (GPIO28_ADC2)
- new net SWR3: R?.1, U?.29 (GPIO22)
- new net SWR4: R?.1, U?.22 (GPIO17)
- new net TUNE: R?.2, SW?.2, U?.24 (GPIO18)
- new net TX+: R?.2
- new net TX0: U?.1 (GPIO0)
- new net TX_GND: J?.2, Q?.1 (B), R?.1
- new net TX_INH: J?.8
- new net _RF_IN: K?.5, K?.6
Other:
- moved on the sheet: K?

Commit message: update
Parts:
- removed J?: USB_B, symbol Connector:USB_B
- added C30: 100nF, Capacitor_SMD:C_0805_2012Metric, symbol Device:C
- added C31, C32, C33, C34: 1uF, Capacitor_SMD:C_0805_2012Metric, symbol Device:C
- added C51, C52, C53, C54: 10nF, Capacitor_SMD:C_0805_2012Metric, symbol Device:C
- added D16: >2.5, LED_THT:LED_D3.0mm_Horizontal_O3.81mm_Z2.0mm, symbol Device:LED
- added D23, D24: PRTR5V0U2X, Package_TO_SOT_SMD:SOT-143, symbol Power_Protection:PRTR5V0U2X
- added D26, D27: BAT54W, Package_TO_SOT_SMD:SOT-323_SC-70, symbol Diode:BAT54W
- added D28, D29: BZX84C5V1, Diode_SMD:D_SOT-23_ANK, symbol Diode:BZX84Cxx
- added J5: USB_A, symbol Connector:USB_A
- added L10, L9: 100uH, Inductor_SMD:L_12x12mm_H8mm, symbol Device:L_Ferrite
- added Q18: 2N2222A_SMD, Package_TO_SOT_SMD:TSOT-23, symbol Transistor:2N2222A_SMD
- added Q20, Q21: BSS138, Package_TO_SOT_SMD:SOT-23, symbol Transistor_FET:BSS138
- added R33, R38, R40, R42, R43, R53, R54, R55, R56, R61, R62: 10k, Resistor_SMD:R_0805_2012Metric, symbol Device:R
- added R34: 1.5k, Resistor_SMD:R_0805_2012Metric, symbol Device:R
- added R35: 1k, Resistor_SMD:R_0805_2012Metric, symbol Device:R
- added R47, R48, R49, R50: 0, Resistor_SMD:R_0805_2012Metric, symbol Device:R
- added R57, R60: 68k, Resistor_SMD:R_0805_2012Metric, symbol Device:R
- added R58, R59: 51, Resistor_SMD:R_0805_2012Metric, symbol Device:R
- added T1: 2_x_1:10, symbol Trafo:2_x_1{colon}10
- added U3: ATmega328-A, Package_QFP:TQFP-32_7x7mm_P0.8mm, symbol MCU_Microchip_ATmega:ATmega328-A
- C1, C12, C16, C17, C2, C23, C24, C26, C27, C28, C29, C3, C37, C39, C40, C42, C44, C7, C8: renamed from C?; value 100n -> 100nF; footprint (none) -> Capacitor_SMD:C_0805_2012Metric; Orderd (none) -> Y
- C10, C13, C14, C20, C21, C9: renamed from C?; footprint (none) -> Capacitor_SMD:C_0805_2012Metric; Orderd (none) -> Y
- C18, C19, C5, C6: renamed from C?; Orderd (none) -> Y
- C38, C41, C43: renamed from C?; footprint (none) -> Capacitor_SMD:CP_Elec_6.3x5.4; Orderd (none) -> Y
- C47, C48: renamed from C?; value 10u -> 10uF; Orderd (none) -> Y
- D1, D10, D11, D12, D13, D14, D2, D21, D22, D25, D3, D4, D5, D6, D7, D8, D9: renamed from D?; Orderd (none) -> Y
- D15, D17, D18, D19, D20: renamed from D?; footprint (none) -> LED_THT:LED_D3.0mm_Horizontal_O3.81mm_Z2.0mm
- F1, F2: renamed from F?; footprint (none) -> Fuse:Fuse_1206_3216Metric
- J4: renamed from J?; footprint (none) -> Connector_PinHeader_2.54mm:PinHeader_1x03_P2.54mm_Vertical; Orderd (none) -> Y
- J8: renamed from J?; footprint (none) -> Connector_USB:USB_B_OST_USB-B1HSxx_Horizontal; Orderd (none) -> Y
- JP1, JP2: renamed from JP?; footprint (none) -> Jumper:SolderJumper-2_P1.3mm_Open_TrianglePad1.0x1.5mm
- L4, L5: renamed from L?; value 100u -> 100uH; footprint (none) -> Inductor_SMD:L_12x12mm_H8mm; Orderd (none) -> Y
- LNA1: renamed from LNA; footprint (none) -> Resistor_SMD:R_0805_2012Metric; Orderd (none) -> Y
- Q1, Q10, Q11, Q12, Q13, Q14, Q15, Q16, Q17, Q19, Q2, Q3, Q4, Q5, Q6, Q7, Q8, Q9: renamed from Q?; Orderd (none) -> Y
- R1, R10, R11, R12, R13, R14, R15, R16, R17, R18, R19, R2, R20, R21, R22, R23, R24, R25, R26, R27, R28, R29, R3, R30, R31, R4, R44, R45, R46, R5, R51, R52, R6, R7, R8, R9: renamed from R?; footprint (none) -> Resistor_SMD:R_0805_2012Metric; Orderd (none) -> Y
- R32, R36, R37, R39, R41: renamed from R?; value R -> 1.5k; footprint (none) -> Resistor_SMD:R_0805_2012Metric; Orderd (none) -> Y
- SW1, SW2, SW3: renamed from SW?; footprint (none) -> Button_Switch_THT:SW_Tactile_SPST_Angled_PTS645Vx83-2LFS
- U1, U4, U6: renamed from U?; Orderd (none) -> Y
- U5: renamed from U?; footprint SO16 -> Package_SO:SOP-16_3.9x9.9mm_P1.27mm; Orderd (none) -> Y
- Y1: renamed from Y?; value Crystal -> 12MHz; Orderd (none) -> Y
- gave numbers to parts that had none: 38
Connections:
- net +12V: now also C10.1, C5.1, C6.1, C9.1, U1.3 (VI), U2.3 (VI), Q18.3 (C)
- net +3.3V: now also R53.1, R54.1
- net +5P: now also D23.4 (VCC), D24.4 (VCC), J5.1 (VBUS)
- net +5V: now also C30.1, R55.1, R56.1, U3.4 (VCC), U3.6 (VCC)
- net +5VA: now also U3.18 (AVCC)
- net AVSS: now also J6.6, C30.2, C31.2, C32.2, C33.2, C34.2, C51.2, C52.1, C53.1, C54.1, D16.1 (K), D23.1 (GND), D24.1 (GND), D28.1 (A), D29.1 (A), J5.4 (GND), J5.5 (Shield), R35.2, R43.2, R58.2, R59.1, R61.2, R62.2, T1.3, T1.6, U3.21 (GND), U3.3 (GND), U3.5 (GND)
- net C1+: now also U3.28 (PC5); no longer U4.11 (GPIO8)
- net C2+: now also U3.30 (PD0); no longer U4.12 (GPIO9)
- net C3+: now also U3.31 (PD1); no longer U4.14 (GPIO10)
- net C4+: now also U3.32 (PD2); no longer U4.15 (GPIO11)
- net C5+: now also U3.1 (PD3); no longer U4.16 (GPIO12)
- net FWD: now also C53.2, D28.3 (K), R57.2, R61.1, U3.22 (ADC7); no longer U4.31 (GPIO26_ADC0)
- net IO+: now also U3.27 (PC4); no longer U4.17 (GPIO13)
- net L1+: now also U3.26 (PC3); no longer U4.4 (GPIO2)
- net L1_I: now also T1.2, T1.8
- net L2+: now also U3.25 (PC2); no longer U4.5 (GPIO3)
- net L3+: now also U3.12 (PB0); no longer U4.6 (GPIO4)
- net L4+: now also U3.11 (PD7); no longer U4.7 (GPIO5)
- net L5+: now also U3.10 (PD6); no longer U4.9 (GPIO6)
- net L6+: now also U3.9 (PD5); no longer U4.10 (GPIO7)
- net REV: now also C54.2, D29.3 (K), R60.2, R62.1, U3.19 (ADC6); no longer U4.32 (GPIO27_ADC1)
- net RF_IN: now also L9.1
- net RST: now also U3.29 (~{RESET}/PC6)
- net RX0: now also R48.1, R50.1
- net SWR3: now also R41.1, U3.14 (PB2); no longer R39.1, U4.29 (GPIO22)
- net TUNE: now also U3.7 (XTAL1/PB6); no longer U4.24 (GPIO18)
- net TX0: now also R47.1, R49.1
- net _RF_IN: now also T1.5
- net TX5: now reaches J6.4
- net TX5: now also Q21.3 (D), R56.2
- net RX5: now reaches J6.5
- net RX5: now also Q20.3 (D), R55.2
- net at U5.7 (DM1): now also D23.2 (I/O1), J5.2 (D-)
- net at U5.8 (DP1): now also D23.3 (I/O2), J5.3 (D+)
- net at J8.3 (D+), U5.10 (DP): now also D24.2 (I/O1)
- net at J8.2 (D-), U5.9 (DM): now also D24.3 (I/O2)
- net SWR1: no longer names the net of U4.20 (GPIO15)
- net SWR1: no longer R36.1
- net SWR2: no longer names the net of U4.34 (GPIO28_ADC2)
- net SWR2: no longer R37.1
- net SWR4: no longer names the net of U4.22 (GPIO17)
- net SWR4: no longer R41.1
- new net: D16.2 (A), R34.2
- new net: C52.2, D27.3 (K), R60.1
- new net: L10.1, L9.2
- new net: C32.1, L10.2, R33.1
- new net: R40.2, R42.2
- new net: D27.1 (A), R59.2, T1.1, T1.7
- new net: D26.1 (A), R58.1, T1.4
- new net: Q18.2 (E), R35.1, R38.2
- new net: C51.1, D26.3 (K), R57.1
- new net: C31.1, U3.20 (AREF)
- new net: C33.1, Q18.1 (B), R33.2
- new net: R38.1, R40.1
- new net ACK: R34.1, U3.8 (XTAL2/PB7)
- new net MISO: R37.1, U3.16 (PB4)
- new net MOSI: R39.1, U3.15 (PB3)
- new net M_SENS: C34.1, R42.1, R43.1, U4.31 (GPIO26_ADC0)
- new net RX3: Q20.1 (G), Q20.2 (S), R47.2, R48.2, R53.2
- new net SCK: R36.1, U3.17 (PB5)
- new net TX3: Q21.1 (G), Q21.2 (S), R49.2, R50.2, R54.2
Other:
- moved on the sheet: C35, C36, C37, C38, C39, C40, C41, C42, C43, C44, C45, C46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
