File: 01_Hardware/ATU-FT891/ATU-FT891.kicad_sch (KiCad schematic)
At the start: 206 parts, among them J1 Conn_Coaxial, J11 Conn_02x03_Counter_Clockwise, J2 Conn_Coaxial, J3 Conn_Coaxial, J4 Conn_01x03_Male, J5 USB_A, J6 Mini-DIN-8, J7 Mini-DIN-6, J8 USB_B, K1 G5V-1, K10 G5V-1, K11 G5V-1, K12 G5V-1, K13 G5V-1, K14 G5V-1, K15 G5V-1, K2 G5V-1, K3 G5V-1, K4 G5V-1, K5 G5V-1, K6 G5V-1, K7 G5V-1, K8 G5V-1, K9 G5V-1, Q1 2N2222A_SMD, Q10 2N2222A_SMD, Q11 2N2222A_SMD, Q12 2N2222A_SMD, Q13 2N2222A_SMD, Q14 2N2222A_SMD, Q15 2N2222A_SMD, Q16 2N2222A_SMD, Q17 2N2222A_SMD, Q19 2N2222A_SMD, Q2 2N2222A_SMD, Q20 BSS138, Q21 BSS138, Q3 2N2222A_SMD, Q4 2N2222A_SMD, Q5 2N2222A_SMD, Q6 2N2222A_SMD, Q7 2N2222A_SMD, Q8 2N2222A_SMD, Q9 2N2222A_SMD, SW1 TUNE, SW2 RST, SW3 LNA, T1 2_x_1:10, U1 NCP1117-3.3_SOT223, U2 NCP1117-5.0_SOT223, U3 ATmega328-A, U4 Pico, U5 SL2.1A, U6 CM118B, Y1 12MHz

Commit message: remove audio
Parts:
- removed C12, C32, C33, C34, C37, C39, C40, C42, C44, C55: 100nF, Capacitor_SMD:C_0805_2012Metric, symbol Device:C
- removed C35, C36: 0.47uF, Capacitor_SMD:C_0805_2012Metric, symbol Device:C
- removed C38, C41, C43: 100uF, Capacitor_SMD:CP_Elec_6.3x5.4, symbol Device:C_Polarized
- removed C45, C46, C49, C50: 1uF, Capacitor_SMD:C_0805_2012Metric, symbol Device:C
- removed C47, C48: 10uF, Capacitor_SMD:C_0805_2012Metric, symbol Device:C
- removed D21: LNA, LED_THT:LED_D3.0mm_Horizontal_O3.81mm_Z2.0mm, symbol Device:LED
- removed D22, D25: D_Schottky, Diode_SMD:D_SOD-123, symbol Device:D_Schottky
- removed D23, D24: PRTR5V0U2X, Package_TO_SOT_SMD:SOT-143, symbol Power_Protection:PRTR5V0U2X
- removed D6: 1N4148W, Diode_SMD:D_SOD-123, symbol Diode:1N4148W
- removed F1, F2: Polyfuse, Fuse:Fuse_1206_3216Metric, symbol Device:Polyfuse
- removed J4: Conn_01x03_Male, Connector_PinHeader_2.54mm:PinHeader_1x03_P2.54mm_Vertical, symbol Connector:Conn_01x03_Male
- removed J5: USB_A, Connectors:USB, symbol Connector:USB_A
- removed J7: Mini-DIN-6, Connectors:Mini-DIN6, symbol Connector:Mini-DIN-6
- removed J8: USB_B, Connector_USB:USB_B_OST_USB-B1HSxx_Horizontal, symbol Connector:USB_B
- removed K1, K10, K11, K12, K13, K14, K15, K2, K3, K4, K5, K6, K7, K8, K9: G5V-1, Relay_THT:Relay_SPDT_Omron_G5V-1, symbol Relay:G5V-1
- removed LNA1: LNA, LNA:LNA, symbol LNA:LNA
- removed Q10, Q11, Q19, Q6, Q7: 2N2222A_SMD, Package_TO_SOT_SMD:TSOT-23, symbol Transistor:2N2222A_SMD
- removed R12, R15, R18, R19, R52: 10k, Resistor_SMD:R_0805_2012Metric, symbol Device:R
- removed R46: 1k, Resistor_SMD:R_0805_2012Metric, symbol Device:R
- removed R51: 1.5k, Resistor_SMD:R_1206_3216Metric, symbol Device:R
- removed SW3: LNA, Button_Switch_THT:SW_Tactile_SPST_Angled_PTS645Vx83-2LFS, symbol Switch:SW_Push
- removed U4: Pico, PICO:RPi_Pico_SMD_TH, symbol RPi:Pico
- removed U5: SL2.1A, Package_SO:SOP-16_3.9x9.9mm_P1.27mm, symbol SL2.1:SL2.1A
- removed U6: CM118B, Package_QFP:LQFP-48_7x7mm_P0.5mm, symbol CM118B:CM118B
- removed Y1: 12MHz, symbol Device:Crystal
- added J4: Conn_01x04, symbol Connector_Generic:Conn_01x04
- added K1, K10, K11, K12, K13, K14, K2, K3, K4, K5, K6, K7, K8: ~, HRS1H-S-DC12V:HRS1H-S-DC12V, symbol HRS1H-S-DC12V:HRS1H-S-DC12V
- R11: value 100k -> 10k
Connections:
- net TX+ is gone; now on net TX_GND: R6.2
- net _RF_IN is gone; now on net RF_IN: T1.5
- net +12V: now also K1.A1, K10.A1, K11.A1, K12.A1, K13.A1, K14.A1, K2.A1, K3.A1, K4.A1, K5.A1, K6.A1, K7.A1, K8.A1
- net +3.3V: now also J4.1 (Pin_1)
- net +5V: now also R11.1
- net ANT_OUT: now also K13.14, K6.12
- net C1_OC: now also K7.A2
- net C2_OC: now also K8.A2
- net C3_OC: now also K10.A2
- net C4_OC: now also K11.A2
- net C5_OC: now also K12.A2
- net C_I: now also K10.11, K11.11, K12.11, K13.11, K7.11, K8.11
- net IO_OC: now also K13.A2
- net L1_I: now also K1.11, K13.12
- net L1_OC: now also K1.A2
- net L2_OC: now also K2.A2
- net L3_OC: now also K3.A2
- net L4_OC: now also K4.A2
- net L5_OC: now also K5.A2
- net L6_OC: now also K6.A2
- net RF_IN: now also K14.11
- net RX0: now also J4.3 (Pin_3)
- net SDR_OUT: now also K14.14
- net TX: now also K14.A2
- net TX0: now also J4.2 (Pin_2)
- net TX_GND: now also R11.2
- net at L7.1, L8.2: now also K5.12, K6.11
- net at L6.1, L7.2: now also K4.12, K5.11
- net at L1.1, L2.2: now also K1.12, K2.11
- net at C4.1: now also K7.14
- net at C11.1: now also K8.14
- net at C25.1: now also K12.14
- net at C15.1: now also K10.14
- net at L3.1, L6.2: now also K3.12, K4.11
- net at L2.1, L3.2: now also K2.12, K3.11
- net at C22.1: now also K11.14
- net AVSS renamed GND
- net GND: now also J4.4 (Pin_4); no longer R11.2
Other:
- note added: "ATMEGA328 + ISP"
- note added: "Back IO"
- note added: "Front IO"
- note added: "Relais"
- note added: "Relais "Drivers""
- note added: "SWR Bridge"
- note added: "USB + Soundcard"
- note added: "Voltage Regulators: 5V, 3V3, 3V6?"
- moved on the sheet: C1, C10, C11, C13, C14, C15, C16, C17, C18, C19, C2, C20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

Commit message: reorg
Other:
- note removed: "USB + Soundcard"
Changed lines of the file:
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@@
-    (effects (font (size 2.54 2.54) bold) (justify left bottom))
-  )
-  (text "USB + Soundcard" (at 391.16 20.32 0)
     (effects (font (size 2.54 2.54) bold) (justify left bottom))
   )
